File: Display_4inch.kicad_sch (KiCad schematic)
At the start: 8 parts

Commit message: data refresh
Parts:
- removed C?: 0.1uF, symbol Device:C
- removed C?: 0.33uF, symbol Device:C
- removed J?: Screw_Terminal_01x05, symbol Connector:Screw_Terminal_01x05
- removed U?: LM7805_TO220, Package_TO_SOT_THT:TO-220-3_Vertical, symbol Regulator_Linear:LM7805_TO220
- removed U?: AMS1117-3.3, Package_TO_SOT_SMD:SOT-223-3_TabPin2, symbol Regulator_Linear:AMS1117-3.3
- added C? (x2): 100nF, symbol Device:C
- added C?: 10uF, symbol Device:C
- added J?: Screw_Terminal_01x05, symbol Connector:Screw_Terminal_01x05
- added R?: R, symbol Device:R
- added SW?: SW_SPDT, symbol Switch:SW_SPDT
Connections:
- net GND: now also U?.5 (VSS/VSSA), C?.2, C?.2, C?.2, J?.2 (Pin_2), SW?.1 (A)
- net GND_RS232: now also J?.5 (Pin_5)
- net RX: now also J?.3 (Pin_3)
- net TX: now also J?.4 (Pin_4)
- net at U?.19 (PA15/PA14-BOOT0): now also R?.1
- net +3V3: now reaches U?.4 (VDD/VDDA)
- net +3V3: now also C?.1, C?.1, SW?.3 (C)
- net NRST: now reaches U?.6 (NRST)
- net NRST: now also C?.1
- new net: R?.2, SW?.2 (B)
- new net +12V: J?.1 (Pin_1)
Other:
- added sheet Power Source (Power_Source.kicad_sch)
- note removed: "Borne 2EDGRC-5,0 Macho 5P 90º"
- note removed: "Power loss in 7805 We have already discussed above that this type of voltage regulators are known as linear voltage regulator. They drop voltage and losses them in the form of heat. Suppose we provide 12v 0.5A input to 7805 IC that has an output of 5v 0.5A. So the voltage drop made by IC will be 7v. We know, Power (P) = Voltage ( V ) x Current ( I ) Power loss = 7 x 0.5 = 3.5 W Input power = 12 x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"
- note removed: "borne-2edgk-5-0-femea-5p"
- moved on the sheet: U?, U?A, U?B

Commit message: data refresh
Parts:
- removed J?: Screw_Terminal_01x05, symbol Connector:Screw_Terminal_01x05
- added C?: 0.1uF, symbol Device:C
- added D? (x3): LED, symbol Device:LED
Connections:
- net GND: now also U?.15, C?.2
- net at U?.16: now also C?.1
- net Tx LED: now reaches U?.10 (PA3)
- net Tx LED: now also D?.2 (A)
- net Debug LED: now reaches U?.11 (PA4)
- net Debug LED: now also D?.2 (A)
- net Rx LED: now reaches U?.9 (PA2)
- net Rx LED: now also D?.2 (A)
Other:
- added sheet Connectors (Connectors.kicad_sch)
- note removed: "12v / 1A"
- moved on the sheet: C?, U?A, U?B

Commit message: Defines of USART1 pins
Connections:
- net Rx_USART1: now reaches U?.1 (PB7/PB8)
- net Tx_USART1: now reaches U?.20 (PB3/PB4/PB5/PB6)
Other:
- note added: "pin 20 = Tx USART1 = PB6 Pin 1 = Rx USART1 = PB7"
Changed lines of the file:
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@@
+    (stroke (width 0) (type default) (color 0 0 0 0))
+  )
+  (wire (pts (xy 128.905 76.2) (xy 130.81 76.2))
     (stroke (width 0) (type default) (color 0 0 0 0))
   )
@@
     (stroke (width 0) (type default) (color 0 0 0 0))
   )
+  (wire (pts (xy 128.905 73.66) (xy 130.81 73.66))
+    (stroke (width 0) (type default) (color 0 0 0 0))
+  )
   (wire (pts (xy 130.175 101.6) (xy 143.51 101.6))
     (stroke (width 0) (type default) (color 0 0 0 0))
@@
     (stroke (width 0) (type default) (color 0 0 0 0))
   )
+  (text "pin 20 = Tx USART1 = PB6\nPin 1  = Rx USART1 = PB7" (at 82.55 60.96 0)
+    (effects (font (size 1.27 1.27)) (justify left bottom))
+  )
+  (label "Tx_USART1" (at 130.81 73.66 0)
+    (effects (font (size 1.27 1.27)) (justify left bottom))
+  )
+  (label "Rx_USART1" (at 130.81 76.2 0)
+    (effects (font (size 1.27 1.27)) (justify left bottom))
+  )
   (label "Debug LED" (at 62.23 81.28 180)
